File: hw/SaL_Frostburn-v1.5/SaLFrostburn.brd (EAGLE design)
At the start: 72.6 x 19.7 mm, 96 parts, among them U1 ATSAMD21G-A, U2 CC1120, U3 ADXL345, U4 gps, Y1 32.768kHx, Y3 32MHz

Commit message: minor changes to HW
Parts:
- added U$7: ADXL193, SparkFun-Sensors:ADXL193
Changed lines of the file:
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@@
 <element name="JP5" library="SparkFun-Connectors" package="JST-2-SMD-VERT" value="" x="-0.635" y="9.779" rot="MR270"/>
 <element name="STANDOFF4" library="SparkFun-Electromechanical" package="STAND-OFF" value="STAND-OFF" x="65.405" y="2.667"/>
+<element name="U$7" library="SparkFun-Sensors" package="ADXL193" value="ADXL193" x="57.15" y="3.81" rot="MR90"/>
 </elements>
 <signals>
